File: welder.kicad_sch (KiCad schematic)
At the start: 13 parts, among them J1 48 VDC INPUT, Q1 Q_NIGBT_GCE, Q2 Q_NIGBT_GCE, Q3 Q_NIGBT_GCE, Q4 Q_NIGBT_GCE, U1 R-78E15-0.5, U2 R-78E3.3-0.5, U3 MIC4604YM, U4 MIC4604YM

Commit message: updated power supplies
Parts:
- removed U1: R-78E15-0.5, Converter_DCDC:Converter_DCDC_RECOM_R-78E-0.5_THT, symbol Regulator_Switching:R-78E15-0.5
- added C5: 2.2 uF, symbol Device:C
- added C6, C8: 0.1 uF, symbol Device:C
- added C7: 10 uF, symbol Device:C
- added C9: 22 uF, symbol Device:C
- added L1: 12 uH, Inductor_SMD:L_Bourns_SRN6045TA, symbol Device:L
- added U1: RPMH15-0.5, Converter_DCDC:Converter_DCDC_RECOM_RPMx.x-x.0, symbol Converter_DCDC:RPM5.0-3.0
Connections:
- net -VDC is gone; now on net GND: C1.1, C2.1, J1.2 (Pin_2), Q2.3 (E), Q4.3 (E), U3.7 (VSS), U4.7 (VSS)
- net +15V: now also U2.1 (IN), C6.1, C9.1, U1.A5 (+VOUT), U1.B5 (+VOUT), U1.C5 (Sense)
- net +3V3: now also C8.1
- net GND: now reaches U2.2 (GND)
- net GND: now also C5.2, C6.2, C7.2, C8.2, C9.2, U1.A3 (GND), U1.A4 (GND), U1.B1 (GND), U1.B2 (GND), U1.B3 (GND), U1.B4 (GND), U1.C2 (GND), U1.C3 (GND), U1.C4 (GND), U1.D2 (GND), U1.D3 (GND), U1.D4 (GND), U1.D5 (GND), U1.E3 (GND), U1.E4 (GND)
- net +VDC renamed +48V
- net +48V: now also C5.1, L1.1
- new net: C7.1, L1.2, U1.A1 (+VIN), U1.A2 (+VIN)
Other:
- moved on the sheet: J1, U2
