File: board/welder.kicad_pcb (KiCad board)
At the start: 2 copper layers, 66 x 66 mm, 48 parts, among them J1 VIN, J2 Conn_01x10, J3 Barrel_Jack_Switch, J4 USB_B, J5 POS, J6 NEG, J7 GND, Q1 Q_NIGBT_GCE, Q2 Q_NIGBT_GCE, Q3 Q_NIGBT_GCE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

Commit message: added display, fixed up field names, updated board
Parts:
- added D6: FML340A-W, Diode_SMD:D_SMA, F.Cu at (109.6, -0.72)
- added Q5: Q_NPN_BEC, Package_TO_SOT_SMD:SOT-23, F.Cu at (223.5, 149.9)
- added Q6: Q_NPN_BEC, Package_TO_SOT_SMD:SOT-23, F.Cu at (223.5, 145.4)
- added Q7: Q_NPN_BEC, Package_TO_SOT_SMD:SOT-23, F.Cu at (244.3, 93.6)
- added Q8: Q_NPN_BEC, Package_TO_SOT_SMD:SOT-23, F.Cu at (249.2, 93.6)
- added R10: 220, Resistor_SMD:R_0805_2012Metric, F.Cu at (262.7, 92.8)
- added R11: 220, Resistor_SMD:R_0805_2012Metric, F.Cu at (253.9, 92.8)
- added R12: 470, Resistor_SMD:R_0805_2012Metric, F.Cu at (271.5, 92.8)
- added R13: 470, Resistor_SMD:R_0805_2012Metric, F.Cu at (228.2, 144.7)
- added R14: 470, Resistor_SMD:R_0805_2012Metric, F.Cu at (253.9, 95.8)
- added R15: 470, Resistor_SMD:R_0805_2012Metric, F.Cu at (244.1, 97.3)
- added R4: 220, Resistor_SMD:R_0805_2012Metric, F.Cu at (258.3, 92.8)
- added R5: 220, Resistor_SMD:R_0805_2012Metric, F.Cu at (275.9, 92.8)
- added R6: 220, Resistor_SMD:R_0805_2012Metric, F.Cu at (258.3, 95.8)
- added R7: 220, Resistor_SMD:R_0805_2012Metric, F.Cu at (244.1, 100.2)
- added R8: 220, Resistor_SMD:R_0805_2012Metric, F.Cu at (267.1, 92.8)
- added R9: 220, Resistor_SMD:R_0805_2012Metric, F.Cu at (248.5, 97.3)
- added U8: LTC-5723HR, Display_7Segment:CA56-12EWA, F.Cu at (224.0, 110.9)
- C11, C17, C18, C5, C9: footprint Capacitor_SMD:C_0603_1608Metric -> Capacitor_SMD:C_0805_2012Metric
- FB1: value Ferrite_Bead -> FerriteBead
- J2: footprint Connector_PinHeader_1.27mm:PinHeader_2x05_P1.27mm_Horizontal -> Connector_PinHeader_1.27mm:PinHeader_2x05_P1.27mm_Vertical
- R1, R2: footprint Resistor_SMD:R_0603_1608Metric -> Resistor_SMD:R_0805_2012Metric
- moved J7 165.0 mm to (12.7, 53.3)
- moved J1 149.3 mm to (12.7, 12.7)
- moved C20 132.8 mm to (223.5, 33.0), turned to -90 degrees
- moved J5 91.7 mm to (251.5, 12.7)
- moved J6 84.1 mm to (251.5, 53.3)
- moved L1 51.6 mm to (144.8, 12.7)
Connections:
- U1 pad 13: unconnected-(U1-Pad13) -> /DIG3_EN
- U1 pad 14: unconnected-(U1-Pad14) -> /DIG4_EN
- U1 pad 17: unconnected-(U1-Pad17) -> /DIG1_EN
- U1 pad 18: unconnected-(U1-Pad18) -> /DIG2_EN
- U1 pad 19: unconnected-(U1-Pad19) -> /A
- U1 pad 20: unconnected-(U1-Pad20) -> /B
- U1 pad 21: unconnected-(U1-Pad21) -> /C
- U1 pad 22: unconnected-(U1-Pad22) -> /D
- U1 pad 23: unconnected-(U1-Pad23) -> /E
- U1 pad 24: unconnected-(U1-Pad24) -> /F
- U1 pad 25: unconnected-(U1-Pad25) -> /G
- U1 pad 27: unconnected-(U1-Pad27) -> /DP

Commit message: Add buttons, update board
Parts:
- added J8: EXT, TerminalBlock_Phoenix:TerminalBlock_Phoenix_MKDS-1,5-3_1x03_P5.00mm_Horizontal, F.Cu at (147.3, 30.5)
- added SW1: INC, Button_Switch_SMD:SW_SPST_PTS645, F.Cu at (221.0, 101.6)
- added SW2: DEC, Button_Switch_SMD:SW_SPST_PTS645, F.Cu at (221.0, 116.8)
- added SW3: SET, Button_Switch_SMD:SW_SPST_PTS645, F.Cu at (172.7, 132.1)
- added SW4: SEL, Button_Switch_SMD:SW_SPST_PTS645, F.Cu at (190.5, 132.1)
- moved D3 225.0 mm to (-61.0, 38.1)
- moved D1 202.1 mm to (-58.4, 81.3)
- moved D4 202.0 mm to (-73.7, 96.5)
- moved D2 192.8 mm to (-63.5, 61.0)
- moved J4 185.3 mm to (19.3, 123.2), turned to 180 degrees
- moved Q2 170.9 mm to (-26.1, 96.5)
- moved U4 158.4 mm to (-38.1, 45.7)
- moved Q1 152.0 mm to (-25.8, 73.5)
- moved U7 145.9 mm to (231.1, 78.7)
- moved Q4 134.4 mm to (-25.8, 55.9)
- moved R3 134.2 mm to (231.1, 66.0)
- moved J2 134.0 mm to (7.62, 139.7)
- moved U3 132.3 mm to (-40.6, 76.8)
- moved Q3 128.7 mm to (-28.3, 37.9)
- moved U6 121.4 mm to (35.6, 121.9), turned to 180 degrees
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Connections:
- U1 pad 1: unconnected-(U1-Pad1) -> /INC
- U1 pad 2: unconnected-(U1-Pad2) -> /DEC
- U1 pad 4: unconnected-(U1-Pad4) -> /SET
- U1 pad 7: unconnected-(U1-Pad7) -> /SEL
- U1 pad 8: unconnected-(U1-Pad8) -> /EXT

Commit message: add heatsinks
Parts:
- added D7: 10A10-T, Diode_THT:D_P600_R-6_P7.62mm_Vertical_AnodeUp, F.Cu at (7.62, -71.1)
- added D8: 10A10-T, Diode_THT:D_P600_R-6_P7.62mm_Vertical_AnodeUp, F.Cu at (7.62, -81.8)
- added HS1: Heatsink_Pad, colinholzman:Ohmite_C60-075, F.Cu at (129.5, -50.5)
- added HS2: Heatsink_Pad, colinholzman:Ohmite_C60-075, F.Cu at (182.5, -50.5)
- added R16: 0, Resistor_SMD:R_0805_2012Metric, F.Cu at (24.2, -85.6)
- added R17: 3.3, Resistor_SMD:R_1206_3216Metric, F.Cu at (-68.1, -1.38)
- added R18: 0, Resistor_SMD:R_0805_2012Metric, F.Cu at (4.50, -64.3)
- added R19: 0, Resistor_SMD:R_0805_2012Metric, F.Cu at (19.8, -85.6)
- added R20: 3.3, Resistor_SMD:R_1206_3216Metric, F.Cu at (-63.7, -1.38)
- added R21: 0, Resistor_SMD:R_0805_2012Metric, F.Cu at (-72.5, -1.38)
- moved Q1 251.7 mm to (187.5, -60.2), turned to 90 degrees
- moved Q2 248.2 mm to (187.5, -29.9), turned to 90 degrees
- moved Q3 187.7 mm to (124.5, -71.2), turned to -90 degrees
- moved Q4 178.7 mm to (124.5, -40.8), turned to -90 degrees
Connections:
- C4 pad 1: /SENSE- -> Net-(C4-Pad1)
- D1 pad 2: Net-(C3-Pad1) -> Net-(D1-Pad2)
- D2 pad 1: Net-(C3-Pad1) -> Net-(D1-Pad2)
- L1 pad 1: Net-(C3-Pad1) -> Net-(D1-Pad2)
- Q1 pad 3: Net-(C3-Pad1) -> Net-(D1-Pad2)
- Q2 pad 2: Net-(C3-Pad1) -> Net-(D1-Pad2)
- U3 pad 3: Net-(Q1-Pad1) -> Net-(R16-Pad1)
- U3 pad 8: Net-(Q2-Pad1) -> Net-(R18-Pad1)
- U4 pad 3: Net-(Q3-Pad1) -> Net-(R19-Pad1)
- U4 pad 4: /SENSE- -> Net-(C4-Pad1)
- U4 pad 8: Net-(Q4-Pad1) -> Net-(R21-Pad1)
